Commit message: feat: 更新夹爪 URDF 为真实 mesh 模型
- 从 reBotArmController_ROS2 项目导入夹爪 mesh 文件
  - gripper_link.STL, gripper_left.STL, gripper_right.STL
- 更新 rebotarm.urdf，使用真实夹爪模型替换简化 box
  - gripper_link (fixed to link6)
  - gripper_finger_left (prismatic, limit 0-0.0715m)
  - gripper_finger_right (mimic left)
- 更新 ros2_controllers.yaml
  - controller_manager update_rate: 100 → 500 Hz
  - arm_controller state_publish_rate: 50 → 200 Hz
  - 添加 gripper_controller 配置
- 更新 relay_node.py
  - 添加 goal 超时机制 (100ms)
  - 轨迹执行时间: 50ms → 20ms
  - 修复 numpy float 类型转换问题
- 更新 relay.yaml
  - max_velocity: 3.0 → 10.0 rad/s
  - publish_rate: 100 → 200 Hz
  - command_timeout: 100ms → 50ms
- 更新 start_gazebo.sh
  - gripper_controller 在 arm_controller 后启动
- 更新 SRDF 和 MoveIt 配置

Co-Authored-By: Claude <noreply@anthropic.com>

File: src/rebotarm_gazebo/urdf/rebotarm.ros2_control.xacro (robot description, xacro)
@@ -65,4 +65,14 @@
       <state_interface name="velocity"/>
     </joint>
+    <joint name="gripper_finger_left_joint">
+      <command_interface name="position">
+        <param name="min">0</param>
+        <param name="max">0.0715</param>
+      </command_interface>
+      <state_interface name="position">
+        <param name="initial_value">0.0</param>
+      </state_interface>
+      <state_interface name="velocity"/>
+    </joint>
   </ros2_control>
   <gazebo>

File: src/rebotarm_gazebo/urdf/rebotarm.urdf (robot description, URDF)
Before this commit: robot reBot-DevArm_fixend, 8 links, 7 joints
Links:
- removed link end_link
- added link gripper_finger_left, mass 0.0423278952416158; collision mesh filename=package://rebotarm_gazebo/meshes/gripper_left.STL; visual mesh filename=package://rebotarm_gazebo/meshes/gripper_left.STL
- added link gripper_finger_right, mass 0.0423278949561274; collision mesh filename=package://rebotarm_gazebo/meshes/gripper_right.STL; visual mesh filename=package://rebotarm_gazebo/meshes/gripper_right.STL
- added link gripper_link, mass 0.181800159145243; collision mesh filename=package://rebotarm_gazebo/meshes/gripper_link.STL; visual mesh filename=package://rebotarm_gazebo/meshes/gripper_link.STL
Joints:
- removed joint end_joint
- added joint gripper_finger_left_joint: type prismatic, parent gripper_link, child gripper_finger_left, origin xyz=-0.042091 2.7531E-05 -1.3031E-05 rpy=0 0 -1.5708, axis 1 0 0, limit lower=0 upper=0.0715 effort=100 velocity=15
- added joint gripper_finger_right_joint: type prismatic, parent gripper_link, child gripper_finger_right, origin xyz=-0.042091 -2.7531E-05 1.3031E-05 rpy=0 0 1.5708, axis 1 0 0, limit lower=0 upper=0.0715 effort=100 velocity=15, mimic joint=gripper_finger_left_joint multiplier=1
- added joint gripper_joint: type fixed, parent link6, child gripper_link, origin xyz=0 0 0.15971 rpy=0 -1.5708 0, axis 0 0 0

File: src/rebotarm_moveit_config/config/rebotarm.ros2_control.xacro (robot description, xacro)
@@ -23,4 +23,5 @@
     <xacro:joint_interface name="joint5" lower="-1.57" upper="1.57"/>
     <xacro:joint_interface name="joint6" lower="-3.14" upper="3.14"/>
+    <xacro:joint_interface name="gripper_finger_left_joint" lower="0" upper="0.0715"/>
   </ros2_control>
 </robot>
