Commit message: feat: 性能优化与诊断工具
- 从臂状态发布频率 50→100 Hz，提升反馈实时性
- relay 发布频率 200→100 Hz，减少 DDS 带宽浪费
- 夹爪 EMA alpha 0.3→0.5，提升响应速度，支持 ROS2 参数动态调整
- 关节增益分离: joint1-3 大电机 / joint4-6 小电机独立配置
- 夹爪 kp/kd 调优: 12/3 → 6/1.5 减少振荡
- CAN 总线速率 500kbps → 1Mbps
- start_jetson.sh 添加 venv 激活
- link2 质量修正 0.383→0.4213 kg
- 新增 debug/ joint4 振动诊断工具包
- 新增 scripts/measure_gripper_range.py 夹爪行程测量

Co-Authored-By: Claude <noreply@anthropic.com>

File: src/rebotarm_gazebo/urdf/rebotarm.urdf (robot description, URDF)
Before this commit: robot reBot-DevArm_fixend, 10 links, 9 joints
Links:
- link link5: mass 0.38300000 -> 0.42130000
