Commit message: feat: 添加手眼标定相机固定关节

File: src/rebotarm_gazebo/urdf/rebotarm.urdf (robot description, URDF)
Before this commit: robot reBot-DevArm_fixend, 10 links, 9 joints
Links:
- added link camera_link
Joints:
- added joint camera_mount_joint: type fixed, parent link6, child camera_link, origin xyz=0.0520 -0.0139 0.0672 rpy=0.0136 1.2829 3.1100

Commit message: fix: make joint4 calibration faults recoverable
Clear the pose fault latch on explicit release and cover the recovery transition. Includes the pending joint4 calibration controller files required to build and test the fix.\n\nRefs #1

File: src/rebotarm_gazebo/urdf/rebotarm.urdf (robot description, URDF)
Before this commit: robot reBot-DevArm_fixend, 11 links, 10 joints
Links:
- link camera_link: mass None -> 0.075

Commit message: tune: 调整夹爪惯性参数
- gripper_link 质量定为 0.4 kg，惯性张量按质量比例缩放，质心同步更新
- gripper_finger_left/right 质量 0.0752 kg，更新质心与惯性张量
- 统一 URDF 换行符为 LF

真实机械臂重力补偿测试表现良好（Jetson，damiao 主机）。

File: src/rebotarm_gazebo/urdf/rebotarm.urdf (robot description, URDF)
Before this commit: robot reBot-DevArm_fixend, 11 links, 10 joints
Links:
- link gripper_finger_left: mass 0.0423278952416158 -> 0.0752
- link gripper_finger_right: mass 0.0423278949561274 -> 0.0752
- link gripper_link: mass 0.181800159145243 -> 0.4

Commit message: fix: restore calibrated wrist camera orientation (#32)

File: src/rebotarm_gazebo/urdf/rebotarm.urdf (robot description, URDF)
Before this commit: robot reBot-DevArm_fixend, 11 links, 10 joints
Joints:
- joint camera_mount_joint: origin xyz=0.0520 -0.0139 0.0672 rpy=0.0136 1.2829 3.1100 -> xyz=0.0520795 -0.0139823 0.0672182 rpy=0.058487598396866 -1.282446543624948 3.076557194400623
