Commit message: feat: 增加夹爪标定与遥操作映射

File: src/plugin/microros_stm32h723_bridge/urdf/rebotarm.arm.micro_ros.xacro (robot description, xacro)
@@ -2,4 +2,5 @@
 <robot xmlns:xacro="http://www.ros.org/wiki/xacro" name="rebotarm_arm">
   <xacro:arg name="gains_file" default="$(find microros_stm32h723_bridge)/config/arm_mit_gains.yaml"/>
+  <xacro:arg name="enable_gripper" default="false"/>
   <xacro:include filename="$(find rebotarm_gazebo)/urdf/rebotarm.urdf"/>
   <ros2_control name="Stm32H723ArmSystem" type="system">
@@ -13,6 +14,13 @@
       <param name="return_duration_ms">3000</param>
       <param name="zero_tolerance">0.03</param>
-      <param name="required_joint_mask">0x3F</param>
+      <xacro:if value="$(arg enable_gripper)">
+        <param name="required_joint_mask">0x7F</param>
+      </xacro:if>
+      <xacro:unless value="$(arg enable_gripper)">
+        <param name="required_joint_mask">0x3F</param>
+      </xacro:unless>
       <param name="gains_file">$(arg gains_file)</param>
+      <param name="gripper_position_scale">-0.008612826752</param>
+      <param name="gripper_position_offset">0.004282757541</param>
     </hardware>
     <joint name="joint1">
@@ -76,4 +84,16 @@
       <command_interface name="effort"/>
     </joint>
+    <xacro:if value="$(arg enable_gripper)">
+      <joint name="gripper_finger_left_joint">
+        <command_interface name="position">
+          <param name="min">0.0</param>
+          <param name="max">0.05</param>
+        </command_interface>
+        <state_interface name="position"/>
+        <state_interface name="velocity"/>
+        <state_interface name="effort"/>
+        <command_interface name="effort"/>
+      </joint>
+    </xacro:if>
   </ros2_control>
 </robot>

Commit message: feat: add opt-in bounded trajectory integral trim
Refs #43. Preserve existing position gates and effort limits; reset trim on controller ownership, MCU reset, fault or stale status.

File: src/plugin/microros_stm32h723_bridge/urdf/rebotarm.arm.micro_ros.xacro (robot description, xacro)
@@ -3,4 +3,6 @@
   <xacro:arg name="gains_file" default="$(find microros_stm32h723_bridge)/config/arm_mit_gains.yaml"/>
   <xacro:arg name="enable_gripper" default="false"/>
+  <xacro:arg name="trajectory_integral_config" default=""/>
+  <xacro:property name="trajectory_integral_config_path" value="$(arg trajectory_integral_config)"/>
   <xacro:include filename="$(find rebotarm_gazebo)/urdf/rebotarm.urdf"/>
   <ros2_control name="Stm32H723ArmSystem" type="system">
@@ -21,4 +23,7 @@
       </xacro:unless>
       <param name="gains_file">$(arg gains_file)</param>
+      <xacro:if value="${trajectory_integral_config_path != ''}">
+        <param name="trajectory_integral_config">${trajectory_integral_config_path}</param>
+      </xacro:if>
       <param name="gripper_position_scale">-0.008612826752</param>
       <param name="gripper_position_offset">0.004282757541</param>

Commit message: refactor: remove experimental hardware integral compensation
Refs #45. Retain gravity feedforward, velocity ownership, effort limits and DISABLE regression coverage.

File: src/plugin/microros_stm32h723_bridge/urdf/rebotarm.arm.micro_ros.xacro (robot description, xacro)
@@ -3,6 +3,4 @@
   <xacro:arg name="gains_file" default="$(find microros_stm32h723_bridge)/config/arm_mit_gains.yaml"/>
   <xacro:arg name="enable_gripper" default="false"/>
-  <xacro:arg name="trajectory_integral_config" default=""/>
-  <xacro:property name="trajectory_integral_config_path" value="$(arg trajectory_integral_config)"/>
   <xacro:include filename="$(find rebotarm_gazebo)/urdf/rebotarm.urdf"/>
   <ros2_control name="Stm32H723ArmSystem" type="system">
@@ -23,7 +21,4 @@
       </xacro:unless>
       <param name="gains_file">$(arg gains_file)</param>
-      <xacro:if value="${trajectory_integral_config_path != ''}">
-        <param name="trajectory_integral_config">${trajectory_integral_config_path}</param>
-      </xacro:if>
       <param name="gripper_position_scale">-0.008612826752</param>
       <param name="gripper_position_offset">0.004282757541</param>
